Commit message: added imu,  tested in gazebo

File: diffbot_description/urdf/diffbot.urdf.xacro (robot description, xacro)
@@ -46,4 +46,8 @@
   </xacro:motor>
   <!-- Sensors -->
+  <xacro:imu_sensor parent_link="base_link"
+                    sensor_prop="${sensor_prop}">
+    <origin xyz="0 0 0" rpy="0 0 0" />
+  </xacro:imu_sensor>
   <xacro:laser prefix="rplidar" parent_link="base_link"
                    sensor_prop="${sensor_prop}"

File: diffbot_description/urdf/include/common_sensors.xacro (robot description, xacro)
@@ -223,5 +223,5 @@
   </gazebo>
   <joint name="imu_joint" type="fixed">
-    <axis xyz="0 1 0" />
+    <axis xyz="0 0 0" />
     <xacro:insert_block name="joint_origin" />
     <parent link="${parent_link}"/>
@@ -240,4 +240,8 @@
       </ros>
       <!-- frame_name ommited, will be "my_link" -->
+      <bodyName>imu_link</bodyName>
+      <frameName>imu_link</frameName>
+      <topicName>imu/data</topicName>
+      <serviceName>imu_service</serviceName>
     </plugin>
     </sensor>

Commit message: slam with rtabmap works fine

File: diffbot_description/urdf/diffbot.urdf.xacro (robot description, xacro)
@@ -46,8 +46,15 @@
   </xacro:motor>
   <!-- Sensors -->
+  <xacro:camera_sensor parent_link="base_link"
+                    sensor_prop="${sensor_prop}"
+                    visualize="false">
+    <origin xyz="0 0 0" rpy="0 0 0" />
+  </xacro:camera_sensor>
+  <!--
   <xacro:imu_sensor parent_link="base_link"
                     sensor_prop="${sensor_prop}">
     <origin xyz="0 0 0" rpy="0 0 0" />
   </xacro:imu_sensor>
+-->
   <xacro:laser prefix="rplidar" parent_link="base_link"
                    sensor_prop="${sensor_prop}"

Commit message: added laser scan for obstacle

File: diffbot_description/urdf/diffbot.urdf.xacro (robot description, xacro)
@@ -49,5 +49,5 @@
                     sensor_prop="${sensor_prop}"
                     visualize="false">
-    <origin xyz="0 0 0" rpy="0 0 0" />
+    <origin xyz="0.080 0 0.090" rpy="0 0 0" />
   </xacro:camera_sensor>
   <!--

File: diffbot_description/urdf/include/common_sensors.xacro (robot description, xacro)
@@ -49,5 +49,5 @@
     <parent link="${parent_link}"/>
     <child link="${prefix}_laser_link"/>
-    <origin xyz="${sensor_prop['laser']['dx']} ${sensor_prop['laser']['dy']} ${sensor_prop['laser']['dz']}" rpy="0 0 ${pi}"/>
+    <origin xyz="${sensor_prop['laser']['dx']} ${sensor_prop['laser']['dy']} ${sensor_prop['laser']['dz']}" rpy="0 0 0"/>
     <axis xyz="0 1 0" />
   </joint>
@@ -127,5 +127,5 @@
   </gazebo>
   <joint name="camera_joint" type="fixed">
-    <axis xyz="0 1 0" />
+    <axis xyz="0 0 0" />
     <xacro:insert_block name="joint_origin" />
     <parent link="${parent_link}"/>

Commit message: adjust sensors's position

File: diffbot_description/urdf/diffbot.urdf.xacro (robot description, xacro)
@@ -49,5 +49,4 @@
                     sensor_prop="${sensor_prop}"
                     visualize="false">
-    <origin xyz="0.080 0 0.090" rpy="0 0 0" />
   </xacro:camera_sensor>
   <!--

File: diffbot_description/urdf/include/common_sensors.xacro (robot description, xacro)
@@ -15,5 +15,5 @@
     <xacro:if value="${mesh != '' }" >
     <visual>
-      <origin xyz="0 0 0" rpy="0 0 ${pi}"/>
+      <origin xyz="0 0 0" rpy="0 0 0"/>
       <geometry>
         <mesh filename="package://${package_name}/meshes/sensors/${mesh}" />
@@ -91,5 +91,5 @@
   </gazebo>
 </xacro:macro>
-<xacro:macro name="camera_sensor" params=" *joint_origin parent_link sensor_prop visualize mesh:='' ">
+<xacro:macro name="camera_sensor" params="parent_link sensor_prop visualize mesh:='' ">
   <link name="camera_link">
     <xacro:if value="${mesh != '' }" >
@@ -127,8 +127,8 @@
   </gazebo>
   <joint name="camera_joint" type="fixed">
-    <axis xyz="0 0 0" />
-    <xacro:insert_block name="joint_origin" />
     <parent link="${parent_link}"/>
     <child link="camera_link"/>
+    <origin xyz="${sensor_prop['camera']['dx']} ${sensor_prop['camera']['dy']} ${sensor_prop['camera']['dz']}" rpy="0 0 0"/>
+    <axis xyz="0 0 0" />
   </joint>
   <gazebo reference="camera_link">

Commit message: add imu "MPU9250"

File: diffbot_description/urdf/diffbot.urdf.xacro (robot description, xacro)
@@ -50,10 +50,8 @@
                     visualize="false">
   </xacro:camera_sensor>
-  <!--
   <xacro:imu_sensor parent_link="base_link"
                     sensor_prop="${sensor_prop}">
     <origin xyz="0 0 0" rpy="0 0 0" />
   </xacro:imu_sensor>
--->
   <xacro:laser prefix="rplidar" parent_link="base_link"
                    sensor_prop="${sensor_prop}"

File: diffbot_description/urdf/include/common_sensors.xacro (robot description, xacro)
@@ -181,5 +181,5 @@
     <xacro:if value="${mesh != '' }" >
       <visual>
-        <origin xyz="0 0 0" rpy="0 0 0"/>
+        <origin xyz="0.085 0 0" rpy="0 0 0"/>
         <geometry>
           <mesh filename="package://${package_name}/meshes/sensors/${mesh}" scale="${sensor_prop['imu']['scale']}" />
@@ -224,10 +224,10 @@
   <joint name="imu_joint" type="fixed">
     <axis xyz="0 0 0" />
-    <origin xyz="0 0 0" rpy="0 0 0"/>
+    <origin xyz="0.085 0 0" rpy="0 0 0"/>
     <parent link="${parent_link}"/>
     <child link="imu_link"/>
   </joint>
   <gazebo reference="imu_link">
-    <sensor type="imu" name="my_imu">
+    <sensor type="imu" name="mpu9250">
     <always_on>true</always_on>
     <!-- Publish at 30 hz -->
@@ -242,5 +242,5 @@
       <bodyName>imu_link</bodyName>
       <frameName>imu_link</frameName>
-      <topicName>imu/data</topicName>
+      <topicName>/rtimulib_node/imu</topicName>
       <serviceName>imu_service</serviceName>
     </plugin>
