Commit message: set origin for imu_joint

File: diffbot_description/urdf/include/common_sensors.xacro (robot description, xacro)
@@ -224,5 +224,5 @@
   <joint name="imu_joint" type="fixed">
     <axis xyz="0 0 0" />
-    <xacro:insert_block name="joint_origin" />
+    <origin xyz="0 0 0" rpy="0 0 0"/>
     <parent link="${parent_link}"/>
     <child link="imu_link"/>

Commit message: localization which wheel and imu

File: diffbot_description/urdf/include/common_sensors.xacro (robot description, xacro)
@@ -224,5 +224,5 @@
   <joint name="imu_joint" type="fixed">
     <axis xyz="0 0 0" />
-    <origin xyz="0.085 0 0" rpy="0 0 0"/>
+    <origin xyz="0.085 0 0" rpy="${pi} 0 0"/>
     <parent link="${parent_link}"/>
     <child link="imu_link"/>

Commit message: use  imu data as NEU

File: diffbot_description/urdf/include/common_sensors.xacro (robot description, xacro)
@@ -178,5 +178,5 @@
   <xacro:property name="mesh"
      value="${sensor_prop['imu']['mesh']}"/>
-  <link name="imu_link">
+  <link name="imu_link_mpu9250">
     <xacro:if value="${mesh != '' }" >
       <visual>
@@ -226,5 +226,5 @@
     <origin xyz="0.085 0 0" rpy="${pi} 0 0"/>
     <parent link="${parent_link}"/>
-    <child link="imu_link"/>
+    <child link="imu_link_mpu9250"/>
   </joint>
   <gazebo reference="imu_link">
